File: pcb/Main_Board_2X-SOLAR_5V-DCDC.brd (EAGLE design)
At the start: 86.4 x 34.4 mm, 75 parts, among them CN5 USBA_FEMALE, IC1 MCP73871, IC2 MCP73871, T2 MMUN2133LT1G, U3 TPS61090RSAR, X1 Solar input, X2 5V output

Commit message: updated layout and BOM
Parts:
- removed U$10: FIDUCIAL, adafruit:FIDUCIAL_1MM
- moved U$3 6.35 mm to (76.2, 31.5)
- moved U$8 4.02 mm to (6.35, 8.89)
Changed lines of the file:
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@@
 <layers>
 <layer number="1" name="Top" color="4" fill="1" visible="yes" active="yes"/>
-<layer number="16" name="Bottom" color="1" fill="1" visible="no" active="yes"/>
+<layer number="16" name="Bottom" color="1" fill="1" visible="yes" active="yes"/>
 <layer number="17" name="Pads" color="2" fill="1" visible="yes" active="yes"/>
 <layer number="18" name="Vias" color="2" fill="1" visible="yes" active="yes"/>
@@
 <layer number="20" name="Dimension" color="15" fill="1" visible="yes" active="yes"/>
 <layer number="21" name="tPlace" color="7" fill="1" visible="yes" active="yes"/>
-<layer number="22" name="bPlace" color="7" fill="1" visible="no" active="yes"/>
+<layer number="22" name="bPlace" color="7" fill="1" visible="yes" active="yes"/>
 <layer number="23" name="tOrigins" color="15" fill="1" visible="yes" active="yes"/>
-<layer number="24" name="bOrigins" color="15" fill="1" visible="no" active="yes"/>
+<layer number="24" name="bOrigins" color="15" fill="1" visible="yes" active="yes"/>
 <layer number="25" name="tNames" color="7" fill="1" visible="yes" active="yes"/>
-<layer number="26" name="bNames" color="7" fill="1" visible="no" active="yes"/>
-<layer number="27" name="tValues" color="7" fill="1" visible="no" active="yes"/>
-<layer number="28" name="bValues" color="7" fill="1" visible="no" active="yes"/>
+<layer number="26" name="bNames" color="7" fill="1" visible="yes" active="yes"/>
+<layer number="27" name="tValues" color="7" fill="1" visible="yes" active="yes"/>
+<layer number="28" name="bValues" color="7" fill="1" visible="yes" active="yes"/>
 <layer number="29" name="tStop" color="7" fill="3" visible="no" active="yes"/>
 <layer number="30" name="bStop" color="7" fill="6" visible="no" active="yes"/>
@@
 <layer number="38" name="bTest" color="7" fill="1" visible="no" active="yes"/>
 <layer number="39" name="tKeepout" color="4" fill="11" visible="yes" active="yes"/>
-<layer number="40" name="bKeepout" color="1" fill="11" visible="no" active="yes"/>
+<layer number="40" name="bKeepout" color="1" fill="11" visible="yes" active="yes"/>
 <layer number="41" name="tRestrict" color="4" fill="10" visible="yes" active="yes"/>
-<layer number="42" name="bRestrict" color="1" fill="10" visible="no" active="yes"/>
+<layer number="42" name="bRestrict" color="1" fill="10" visible="yes" active="yes"/>
 <layer number="43" name="vRestrict" color="2" fill="10" visible="no" active="yes"/>
 <layer number="44" name="Drills" color="7" fill="1" visible="yes" active="yes"/>
@@
 <layer number="50" name="dxf" color="7" fill="1" visible="no" active="yes"/>
 <layer number="51" name="tDocu" color="7" fill="1" visible="yes" active="yes"/>
-<layer number="52" name="bDocu" color="7" fill="1" visible="no" active="yes"/>
+<layer number="52" name="bDocu" color="7" fill="1" visible="yes" active="yes"/>
 <layer number="53" name="tGND_GNDA" color="7" fill="9" visible="no" active="no"/>
 <layer number="54" name="bGND_GNDA" color="1" fill="9" visible="no" active="no"/>
@@
 <text x="66.675" y="2.286" size="1.016" layer="21" ratio="12">EN</text>
 <text x="69.342" y="24.511" size="1.27" layer="22" ratio="12" rot="MR0" align="center">TPS61090 DC Boost</text>
-<text x="69.85" y="27.6098" size="1.016" layer="22" ratio="12" rot="MR0" align="center">iOS 1A Charge Resistors</text>
-<text x="69.342" y="22.479" size="1.27" layer="22" ratio="12" rot="MR0" align="center">5Vout: ~5.2V @ 1A+</text>
-<text x="68.453" y="20.193" size="1.27" layer="22" ratio="12" rot="MR0" align="center">3.2V Low Batt Indicator</text>
+<text x="77.47" y="27.3812" size="1.016" layer="22" ratio="12" rot="MR0">iOS 1A Charge Resistors</text>
+<text x="76.2" y="21.59" size="1.27" layer="22" ratio="12" rot="MR0">5Vout: ~5.2V @ 1A+</text>
+<text x="76.2" y="19.939" size="1.27" layer="22" ratio="12" rot="MR0">3.2V Low Batt Indicator</text>
 <text x="69.469" y="2.286" size="1.016" layer="22" ratio="12" rot="MR90">GND</text>
 <text x="66.929" y="2.413" size="1.016" layer="22" ratio="12" rot="MR90">EN</text>
@@
 <text x="76.962" y="2.413" size="1.016" layer="22" ratio="12" rot="MR90">5Vo</text>
 <text x="64.516" y="2.286" size="1.016" layer="22" ratio="12" rot="MR90">Vbat</text>
-<text x="69.342" y="17.907" size="1.27" layer="22" ratio="12" rot="MR0" align="center">LiPoly 3.7-4.2 V only!</text>
-<text x="68.199" y="15.494" size="1.27" layer="22" ratio="12" rot="MR0" align="center">Vsh:  larger of USB/LiPo</text>
+<text x="76.2" y="18.3642" size="1.27" layer="22" ratio="12" rot="MR0">LiPoly 3.7-4.2 V only!</text>
+<text x="76.2254" y="16.6116" size="1.27" layer="22" ratio="12" rot="MR0">Vsh:  larger of USB/LiPo</text>
 <text x="77.47" y="28.6766" size="1.27" layer="22" ratio="12" rot="MR0">USB: 1A Charge Rate</text>
 <text x="76.708" y="2.413" size="1.016" layer="21" ratio="12">5V</text>
@@
 <element name="C4" library="adafruit" package="E5-13" value="4700uF/10V" x="28.067" y="28.194" smashed="yes">
 <attribute name="NAME" x="26.8224" y="29.7688" size="1.778" layer="25" ratio="10"/>
-<attribute name="VALUE" x="18.669" y="24.257" size="1.778" layer="27" font="vector" ratio="10"/>
+<attribute name="VALUE" x="21.209" y="31.877" size="1.778" layer="27" font="vector" ratio="10"/>
 </element>
 <element name="D1" library="microbuilder" package="SOD-123" value="MBR120VLSFT1G" x="21.844" y="25.527" smashed="yes" rot="R90">
@@
 <attribute name="VALUE" x="8.871" y="17.5704" size="1.27" layer="27" font="vector" ratio="10" rot="R90"/>
 </element>
-<element name="U$3" library="adafruit" package="FIDUCIAL_1MM" value="FIDUCIAL" x="72.39" y="26.416" smashed="yes"/>
+<element name="U$3" library="adafruit" package="FIDUCIAL_1MM" value="FIDUCIAL" x="76.2" y="31.496" smashed="yes"/>
 <element name="U$4" library="microbuilder" package="MOUNTINGHOLE_2.5_PLATED" value="MOUNTINGHOLE2.5" x="3.81" y="3.81"/>
 <element name="U$6" library="microbuilder" package="MOUNTINGHOLE_2.5_PLATED" value="MOUNTINGHOLE2.5" x="3.81" y="30.48"/>
-<element name="U$8" library="adafruit" package="FIDUCIAL_1MM" value="FIDUCIAL" x="2.54" y="7.62"/>
+<element name="U$8" library="adafruit" package="FIDUCIAL_1MM" value="FIDUCIAL" x="6.35" y="8.89"/>
 <element name="IC2" library="adafruit" package="QFN20_4MM" value="MCP73871" x="51.181" y="19.304" smashed="yes">
 <attribute name="NAME" x="49.276" y="21.971" size="0.4064" layer="25"/>
@@
 <element name="C8" library="adafruit" package="E5-13" value="4700uF/10V" x="50.927" y="28.194" smashed="yes">
 <attribute name="NAME" x="49.6824" y="29.7688" size="1.778" layer="25" ratio="10"/>
-<attribute name="VALUE" x="44.069" y="30.607" size="1.778" layer="27" font="vector" ratio="10"/>
+<attribute name="VALUE" x="44.069" y="31.877" size="1.778" layer="27" font="vector" ratio="10"/>
 </element>
 <element name="R17" library="adafruit" package="M0805" value="1K" x="42.926" y="15.748" smashed="yes" rot="R90">
@@
 <attribute name="VALUE" x="34.271" y="11.2204" size="1.27" layer="27" font="vector" ratio="10" rot="R90"/>
 </element>
-<element name="U$10" library="adafruit" package="FIDUCIAL_1MM" value="FIDUCIAL" x="2.54" y="25.654" smashed="yes"/>
 <element name="U$12" library="microbuilder" package="MOUNTINGHOLE_2.5_PLATED" value="MOUNTINGHOLE2.5" x="82.55" y="3.81"/>
 <element name="U3" library="microbuilder" package="PVQFN-16" value="TPS61090RSAR" x="72.531" y="15.286" smashed="yes" rot="R180">
