File: pcb/Main_Board_2X-SOLAR_5V-DCDC.sch (EAGLE design)
At the start: 57 parts, among them M3AB FDMC8030, M4 SI7611DN, M5 FDMC8327L, T2 MMUN2133LT1G, U1 LTC4015EUHFPBFQFN-38_UHF-M, U3 TPS61090RSAR, X1 6V_PV

Commit message: added more components
Parts:
- added C22: 1 uF, microbuilder:CAP_CERAMIC0805-NOOUTLINE
- added RSNSI: KRL3216T4A-M-R004-F-T1, RCT:KRL3216T4A-M-R004-F-T1
Connections:
- net N$10 renamed NTCBIAS
- net N$12 renamed SW_LTC
- net N$2 renamed CCREFM
- net N$6 renamed CCREFP
- net N$8 renamed RT
- net N$9 renamed VC
- removed net N$14: C28.2, U1.CLN
- removed net N$15: C28.1, U1.CLP
- new net CLN: C22.1, C28.2, U1.CLN
- new net CLP: C28.1, RSNSI.3, U1.CLP
- new net N$3: M5.DRAIN, RSNSI.1
- net BAT: now also RSNS.2
- net CSN: now also RSNS.4
- net CSP: now also RSNS.3
- net N$1: now also RSNS.1
- net SYS: now also C22.2, RSNSI.2; no longer M5.DRAIN
Other:
- moved on the sheet: C28
Changed lines of the file:
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@@
 <setting verticaltext="up"/>
 </settings>
-<grid distance="0.1" unitdist="inch" unit="inch" style="lines" multiple="1" display="no" altdistance="0.01" altunitdist="inch" altunit="inch"/>
+<grid distance="0.1" unitdist="inch" unit="inch" style="lines" multiple="1" display="yes" altdistance="0.01" altunitdist="inch" altunit="inch"/>
 <layers>
 <layer number="1" name="Top" color="4" fill="1" visible="no" active="no"/>
@@
 <part name="U$4" library="RCT" deviceset="XAL1010-103ME" device="-103ME"/>
 <part name="RSNS" library="RCT" deviceset="KRL3216T4A-M-R004-F-T1" device=""/>
+<part name="RSNSI" library="RCT" deviceset="KRL3216T4A-M-R004-F-T1" device=""/>
+<part name="C22" library="microbuilder" deviceset="CAP_CERAMIC" device="0805-NOOUTLINE" value="1 uF"/>
 </parts>
 <sheets>
@@
 <instance part="C23" gate="G$1" x="147.32" y="78.74"/>
 <instance part="C24" gate="G$1" x="147.32" y="86.36"/>
-<instance part="C28" gate="G$1" x="137.16" y="127"/>
+<instance part="C28" gate="G$1" x="137.16" y="129.54"/>
 <instance part="M5" gate="G$1" x="124.46" y="152.4" rot="R90"/>
 <instance part="DB" gate="G$1" x="124.46" y="109.22" smashed="yes" rot="R90">
@@
 <instance part="FRAME1" gate="G$2" x="330.2" y="0"/>
 <instance part="U$4" gate="G$1" x="198.12" y="99.06"/>
-<instance part="RSNS" gate="G$1" x="195.58" y="60.96" rot="R90"/>
+<instance part="RSNS" gate="R1" x="205.74" y="58.42" smashed="yes" rot="R270">
+<attribute name="NAME" x="210.82" y="60.198" size="1.27" layer="95"/>
+<attribute name="VALUE" x="210.82" y="56.388" size="1.27" layer="96"/>
+</instance>
+<instance part="RSNSI" gate="R1" x="142.24" y="149.86" smashed="yes">
+<attribute name="NAME" x="139.7" y="146.558" size="1.27" layer="95"/>
+<attribute name="VALUE" x="134.62" y="155.448" size="1.27" layer="96"/>
+</instance>
+<instance part="C22" gate="G$1" x="152.4" y="124.46" smashed="yes" rot="R90">
+<attribute name="NAME" x="151.15" y="129.79" size="1.27" layer="95" font="vector" rot="R180" align="center"/>
+<attribute name="VALUE" x="151.15" y="126.76" size="1.27" layer="96" font="vector" rot="R180" align="center"/>
+</instance>
 </instances>
 <busses>
@@
 <pinref part="U3" gate="G$1" pin="VBAT"/>
 <wire x1="223.52" y1="121.92" x2="215.9" y2="121.92" width="0.1524" layer="91"/>
-<wire x1="215.9" y1="121.92" x2="119.38" y2="121.92" width="0.1524" layer="91"/>
+<wire x1="215.9" y1="121.92" x2="160.02" y2="121.92" width="0.1524" layer="91"/>
+<wire x1="160.02" y1="121.92" x2="119.38" y2="121.92" width="0.1524" layer="91"/>
 <wire x1="292.1" y1="116.84" x2="259.08" y2="116.84" width="0.1524" layer="91"/>
 <pinref part="R45" gate="G$1" pin="2"/>
@@
 <wire x1="165.1" y1="152.4" x2="157.48" y2="152.4" width="0.1524" layer="91"/>
 <junction x="157.48" y="152.4"/>
-<pinref part="C21" gate="G$1" pin="1"/>
+<wire x1="147.32" y1="152.4" x2="149.86" y2="152.4" width="0.1524" layer="91"/>
 <wire x1="149.86" y1="152.4" x2="157.48" y2="152.4" width="0.1524" layer="91"/>
-<junction x="149.86" y="152.4"/>
-<pinref part="M5" gate="G$1" pin="DRAIN"/>
-<wire x1="132.08" y1="152.4" x2="149.86" y2="152.4" width="0.1524" layer="91"/>
 <wire x1="223.52" y1="152.4" x2="243.84" y2="152.4" width="0.1524" layer="91"/>
 <wire x1="243.84" y1="152.4" x2="243.84" y2="121.92" width="0.1524" layer="91"/>
 <junction x="223.52" y="152.4"/>
-</segment>
-</net>
-<net name="N$8" class="0">
+<pinref part="RSNSI" gate="R1" pin="2"/>
+<pinref part="C21" gate="G$1" pin="1"/>
+<junction x="149.86" y="152.4"/>
+<pinref part="C22" gate="G$1" pin="2"/>
+<wire x1="154.94" y1="124.46" x2="160.02" y2="124.46" width="0.1524" layer="91"/>
+<wire x1="160.02" y1="124.46" x2="160.02" y2="121.92" width="0.1524" layer="91"/>
+<junction x="160.02" y="121.92"/>
+</segment>
+</net>
+<net name="RT" class="0">
 <segment>
 <pinref part="U1" gate="A" pin="RT"/>
@@
 </segment>
 </net>
-<net name="N$9" class="0">
+<net name="VC" class="0">
 <segment>
 <pinref part="U1" gate="A" pin="VC"/>
@@
 </segment>
 </net>
-<net name="N$6" class="0">
+<net name="CCREFP" class="0">
 <segment>
 <pinref part="U1" gate="A" pin="CCREFP"/>
@@
 <pinref part="C24" gate="G$1" pin="2"/>
 <wire x1="147.32" y1="83.82" x2="167.64" y2="83.82" width="0.1524" layer="91"/>
-<wire x1="167.64" y1="83.82" x2="167.64" y2="68.58" width="0.1524" layer="91"/>
+<wire x1="167.64" y1="83.82" x2="167.64" y2="63.5" width="0.1524" layer="91"/>
+<pinref part="RSNS" gate="R1" pin="3"/>
+<wire x1="167.64" y1="63.5" x2="205.74" y2="63.5" width="0.1524" layer="91"/>
 </segment>
 </net>
@@
 <wire x1="147.32" y1="76.2" x2="165.1" y2="76.2" width="0.1524" layer="91"/>
 <junction x="147.32" y="76.2"/>
-<wire x1="165.1" y1="53.34" x2="165.1" y2="76.2" width="0.1524" layer="91"/>
+<pinref part="RSNS" gate="R1" pin="4"/>
+<wire x1="205.74" y1="55.88" x2="165.1" y2="55.88" width="0.1524" layer="91"/>
+<wire x1="165.1" y1="55.88" x2="165.1" y2="76.2" width="0.1524" layer="91"/>
 </segment>
 </net>
@@
 <pinref part="U1" gate="A" pin="BATSENS"/>
 <wire x1="134.62" y1="83.82" x2="119.38" y2="83.82" width="0.1524" layer="91"/>
-<label x="137.16" y="68.58" size="1.778" layer="95"/>
 <wire x1="154.94" y1="68.58" x2="162.56" y2="68.58" width="0.1524" layer="91"/>
 <wire x1="162.56" y1="68.58" x2="162.56" y2="50.8" width="0.1524" layer="91"/>
 <junction x="154.94" y="68.58"/>
-<wire x1="162.56" y1="50.8" x2="226.06" y2="50.8" width="0.1524" layer="91"/>
+<wire x1="162.56" y1="50.8" x2="208.28" y2="50.8" width="0.1524" layer="91"/>
 <label x="220.98" y="50.8" size="1.778" layer="95"/>
+<pinref part="RSNS" gate="R1" pin="2"/>
+<wire x1="208.28" y1="50.8" x2="226.06" y2="50.8" width="0.1524" layer="91"/>
+<wire x1="208.28" y1="53.34" x2="208.28" y2="50.8" width="0.1524" layer="91"/>
+<junction x="208.28" y="50.8"/>
 </segment>
 </net>
@@
 </segment>
 </net>
-<net name="N$10" class="0">
+<net name="NTCBIAS" class="0">
 <segment>
 <pinref part="U1" gate="A" pin="NTCBIAS"/>
@@
 </segment>
 </net>
-<net name="N$12" class="0">
+<net name="SW_LTC" class="0">
 <segment>
 <pinref part="M3AB" gate="G$1" pin="S1"/>
@@
 </segment>
 </net>
-<net name="N$14" class="0">
-<segment>
-<pinref part="U1" gate="A" pin="CLN"/>
-<wire x1="119.38" y1="124.46" x2="137.16" y2="124.46" width="0.1524" layer="91"/>
-<pinref part="C28" gate="G$1" pin="2"/>
-</segment>
-</net>
-<net name="N$15" class="0">
-<segment>
+<net name="CLP" class="0">
+<segment>
+<pinref part="C28" gate="G$1" pin="1"/>
+<pinref part="RSNSI" gate="R1" pin="3"/>
+<wire x1="137.16" y1="134.62" x2="137.16" y2="149.86" width="0.1524" layer="91"/>
 <pinref part="U1" gate="A" pin="CLP"/>
 <wire x1="119.38" y1="127" x2="129.54" y2="127" width="0.1524" layer="91"/>
-<wire x1="129.54" y1="127" x2="129.54" y2="132.08" width="0.1524" layer="91"/>
-<wire x1="129.54" y1="132.08" x2="137.16" y2="132.08" width="0.1524" layer="91"/>
-<pinref part="C28" gate="G$1" pin="1"/>
+<wire x1="129.54" y1="127" x2="129.54" y2="134.62" width="0.1524" layer="91"/>
+<wire x1="129.54" y1="134.62" x2="137.16" y2="134.62" width="0.1524" layer="91"/>
+<junction x="137.16" y="134.62"/>
 </segment>
 </net>
@@
 </segment>
 </net>
-<net name="N$2" class="0">
+<net name="CCREFM" class="0">
 <segment>
 <pinref part="RCCREF" gate="G$1" pin="2"/>
@@
 <wire x1="208.28" y1="99.06" x2="203.2" y2="99.06" width="0.1524" layer="91"/>
 <junction x="208.28" y="99.06"/>
-</segment>
-</net>
+<wire x1="208.28" y1="99.06" x2="208.28" y2="66.04" width="0.1524" layer="91"/>
+<pinref part="RSNS" gate="R1" pin="1"/>
+</segment>
+</net>
+<net name="N$3" class="0">
+<segment>
+<pinref part="M5" gate="G$1" pin="DRAIN"/>
+<pinref part="RSNSI" gate="R1" pin="1"/>
+<wire x1="134.62" y1="152.4" x2="132.08" y2="152.4" width="0.1524" layer="91"/>
+</segment>
+</net>
+<net name="CLN" class="0">
+<segment>
+<pinref part="U1" gate="A" pin="CLN"/>
+<wire x1="119.38" y1="124.46" x2="137.16" y2="124.46" width="0.1524" layer="91"/>
+<pinref part="C22" gate="G$1" pin="1"/>
+<pinref part="C28" gate="G$1" pin="2"/>
+<wire x1="137.16" y1="124.46" x2="147.32" y2="124.46" width="0.1524" layer="91"/>
+<wire x1="137.16" y1="127" x2="137.16" y2="124.46" width="0.1524" layer="91"/>
+<junction x="137.16" y="124.46"/>
+</segment>
+</net>

Commit message: Sch/Brd update, added image for silkscreen
Parts:
- added C29: 120 uF, microbuilder:CAP_CERAMIC0805-NOOUTLINE
- added C30: 0.33 uF, microbuilder:CAP_CERAMIC0805-NOOUTLINE
- added CN5: USBA_FEMALE, microbuilder:USB_TYPEAPTHFML
- added R35: 43K, microbuilder:RESISTOR0805_NOOUTLINE
- added R36: 49.9K, microbuilder:RESISTOR0805_NOOUTLINE
- added R37: 75K 1%, microbuilder:RESISTOR0805_NOOUTLINE
- added R38: 49.9K 1%, microbuilder:RESISTOR0805_NOOUTLINE
Connections:
- removed net SYSM5_DRAIN_2: M3AB.D1, U1.SYSM5
- new net D+1: CN5.D+, R37.1, R38.1
- new net D-1: CN5.D-, R35.1, R36.1
- new net N$2: C30.2, U1.SYSM5
- new net N$4: C30.1, M3AB.D1
- net 5.0V: now also CN5.VBUS, R35.2, R37.2
- net CLN: now also RSNSI.4
- net GND: now also C29.1, CN5.GND, R36.2, R38.2
- net SYS: now also C29.2
Changed lines of the file:
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@@
 <setting verticaltext="up"/>
 </settings>
-<grid distance="0.1" unitdist="inch" unit="inch" style="lines" multiple="1" display="yes" altdistance="0.01" altunitdist="inch" altunit="inch"/>
+<grid distance="0.1" unitdist="inch" unit="inch" style="lines" multiple="1" display="no" altdistance="0.01" altunitdist="inch" altunit="inch"/>
 <layers>
 <layer number="1" name="Top" color="4" fill="1" visible="no" active="no"/>
@@
 <part name="RSNSI" library="RCT" deviceset="KRL3216T4A-M-R004-F-T1" device=""/>
 <part name="C22" library="microbuilder" deviceset="CAP_CERAMIC" device="0805-NOOUTLINE" value="1 uF"/>
+<part name="R35" library="microbuilder" deviceset="RESISTOR" device="0805_NOOUTLINE" value="43K"/>
+<part name="R36" library="microbuilder" deviceset="RESISTOR" device="0805_NOOUTLINE" value="49.9K"/>
+<part name="R37" library="microbuilder" deviceset="RESISTOR" device="0805_NOOUTLINE" value="75K 1%"/>
+<part name="R38" library="microbuilder" deviceset="RESISTOR" device="0805_NOOUTLINE" value="49.9K 1%"/>
+<part name="CN5" library="microbuilder" deviceset="USB_TYPEA" device="PTHFML" value="USBA_FEMALE"/>
+<part name="U$56" library="microbuilder" deviceset="5.0V" device=""/>
+<part name="U$57" library="microbuilder" deviceset="5.0V" device=""/>
+<part name="U$58" library="microbuilder" deviceset="5.0V" device=""/>
+<part name="U$67" library="microbuilder" deviceset="GND" device=""/>
+<part name="U$68" library="microbuilder" deviceset="GND" device=""/>
+<part name="U$69" library="microbuilder" deviceset="GND" device=""/>
+<part name="C29" library="microbuilder" deviceset="CAP_CERAMIC" device="0805-NOOUTLINE" value="120 uF"/>
+<part name="U$14" library="microbuilder" deviceset="GND" device=""/>
+<part name="C30" library="microbuilder" deviceset="CAP_CERAMIC" device="0805-NOOUTLINE" value="0.33 uF"/>
 </parts>
 <sheets>
@@
 <instance part="M4" gate="G$1" x="215.9" y="114.3"/>
 <instance part="U$1" gate="G$1" x="187.96" y="142.24"/>
-<instance part="C23" gate="G$1" x="147.32" y="78.74"/>
-<instance part="C24" gate="G$1" x="147.32" y="86.36"/>
+<instance part="C23" gate="G$1" x="147.32" y="78.74" smashed="yes">
+<attribute name="NAME" x="145.03" y="79.99" size="1.27" layer="95" font="vector" rot="R90" align="center"/>
+<attribute name="VALUE" x="153.69" y="81.04" size="1.27" layer="96" font="vector" rot="R180" align="center"/>
+</instance>
+<instance part="C24" gate="G$1" x="147.32" y="86.36" smashed="yes">
+<attribute name="NAME" x="145.03" y="87.61" size="1.27" layer="95" font="vector" rot="R90" align="center"/>
+<attribute name="VALUE" x="153.69" y="88.66" size="1.27" layer="96" font="vector" rot="R180" align="center"/>
+</instance>
 <instance part="C28" gate="G$1" x="137.16" y="129.54"/>
 <instance part="M5" gate="G$1" x="124.46" y="152.4" rot="R90"/>
@@
 </instance>
 <instance part="C22" gate="G$1" x="152.4" y="124.46" smashed="yes" rot="R90">
-<attribute name="NAME" x="151.15" y="129.79" size="1.27" layer="95" font="vector" rot="R180" align="center"/>
-<attribute name="VALUE" x="151.15" y="126.76" size="1.27" layer="96" font="vector" rot="R180" align="center"/>
+<attribute name="NAME" x="153.182" y="127.25" size="1.27" layer="95" font="vector" rot="R180" align="top-right"/>
+<attribute name="VALUE" x="153.182" y="125.236" size="1.27" layer="96" font="vector" rot="R180" align="top-right"/>
+</instance>
+<instance part="R35" gate="G$1" x="281.94" y="180.34"/>
+<instance part="R36" gate="G$1" x="281.94" y="172.72"/>
+<instance part="R37" gate="G$1" x="281.94" y="160.02"/>
+<instance part="R38" gate="G$1" x="281.94" y="152.4"/>
+<instance part="CN5" gate="G$1" x="261.62" y="165.1"/>
+<instance part="U$56" gate="G$1" x="289.56" y="185.42"/>
+<instance part="U$57" gate="G$1" x="289.56" y="165.1"/>
+<instance part="U$58" gate="G$1" x="271.78" y="175.26"/>
+<instance part="U$67" gate="G$1" x="289.56" y="170.18"/>
+<instance part="U$68" gate="G$1" x="289.56" y="147.32"/>
+<instance part="U$69" gate="G$1" x="271.78" y="154.94"/>
+<instance part="C29" gate="G$1" x="236.22" y="149.86" smashed="yes" rot="R180">
+<attribute name="NAME" x="237.002" y="150.11" size="1.27" layer="95" font="vector" rot="R180" align="top-right"/>
+<attribute name="VALUE" x="237.002" y="145.556" size="1.27" layer="96" font="vector" rot="R180" align="top-right"/>
+</instance>
+<instance part="U$14" gate="G$1" x="236.22" y="139.7"/>
+<instance part="C30" gate="G$1" x="137.16" y="119.38" smashed="yes" rot="R270">
+<attribute name="NAME" x="136.378" y="119.13" size="1.27" layer="95" font="vector" align="top-right"/>
+<attribute name="VALUE" x="147.808" y="119.112" size="1.27" layer="96" font="vector" align="top-right"/>
 </instance>
 </instances>
@@
 <junction x="187.96" y="144.78"/>
 </segment>
+<segment>
+<pinref part="R36" gate="G$1" pin="2"/>
+<wire x1="287.02" y1="172.72" x2="289.56" y2="172.72" width="0.1524" layer="91"/>
+<pinref part="U$67" gate="G$1" pin="GND"/>
+</segment>
+<segment>
+<pinref part="R38" gate="G$1" pin="2"/>
+<wire x1="287.02" y1="152.4" x2="289.56" y2="152.4" width="0.1524" layer="91"/>
+<wire x1="289.56" y1="152.4" x2="289.56" y2="149.86" width="0.1524" layer="91"/>
+<pinref part="U$68" gate="G$1" pin="GND"/>
+</segment>
+<segment>
+<pinref part="CN5" gate="G$1" pin="GND"/>
+<wire x1="271.78" y1="160.02" x2="271.78" y2="157.48" width="0.1524" layer="91"/>
+<pinref part="U$69" gate="G$1" pin="GND"/>
+</segment>
+<segment>
+<pinref part="C29" gate="G$1" pin="1"/>
+<pinref part="U$14" gate="G$1" pin="GND"/>
+<wire x1="236.22" y1="142.24" x2="236.22" y2="144.78" width="0.1524" layer="91"/>
+</segment>
 </net>
 <net name="SW" class="0">
@@
 <wire x1="330.2" y1="166.37" x2="322.58" y2="166.37" width="0.1524" layer="91"/>
 <pinref part="JP10" gate="A" pin="8"/>
+</segment>
+<segment>
+<pinref part="R35" gate="G$1" pin="2"/>
+<pinref part="U$56" gate="G$1" pin="5.0V"/>
+<wire x1="287.02" y1="180.34" x2="289.56" y2="180.34" width="0.1524" layer="91"/>
+<wire x1="289.56" y1="180.34" x2="289.56" y2="182.88" width="0.1524" layer="91"/>
+</segment>
+<segment>
+<pinref part="R37" gate="G$1" pin="2"/>
+<pinref part="U$57" gate="G$1" pin="5.0V"/>
+<wire x1="287.02" y1="160.02" x2="289.56" y2="160.02" width="0.1524" layer="91"/>
+<wire x1="289.56" y1="160.02" x2="289.56" y2="162.56" width="0.1524" layer="91"/>
+</segment>
+<segment>
+<pinref part="CN5" gate="G$1" pin="VBUS"/>
+<pinref part="U$58" gate="G$1" pin="5.0V"/>
+<wire x1="271.78" y1="170.18" x2="271.78" y2="172.72" width="0.1524" layer="91"/>
 </segment>
 </net>
@@
 <wire x1="147.32" y1="152.4" x2="149.86" y2="152.4" width="0.1524" layer="91"/>
 <wire x1="149.86" y1="152.4" x2="157.48" y2="152.4" width="0.1524" layer="91"/>
-<wire x1="223.52" y1="152.4" x2="243.84" y2="152.4" width="0.1524" layer="91"/>
+<wire x1="223.52" y1="152.4" x2="236.22" y2="152.4" width="0.1524" layer="91"/>
+<wire x1="236.22" y1="152.4" x2="243.84" y2="152.4" width="0.1524" layer="91"/>
 <wire x1="243.84" y1="152.4" x2="243.84" y2="121.92" width="0.1524" layer="91"/>
 <junction x="223.52" y="152.4"/>
@@
 <wire x1="160.02" y1="124.46" x2="160.02" y2="121.92" width="0.1524" layer="91"/>
 <junction x="160.02" y="121.92"/>
+<pinref part="C29" gate="G$1" pin="2"/>
+<junction x="236.22" y="152.4"/>
 </segment>
 </net>
@@
 <pinref part="RNTCBIAS" gate="G$1" pin="2"/>
 <wire x1="124.46" y1="78.74" x2="124.46" y2="76.2" width="0.1524" layer="91"/>
-</segment>
-</net>
-<net name="SYSM5_DRAIN_2" class="0">
-<segment>
-<pinref part="U1" gate="A" pin="SYSM5"/>
-<pinref part="M3AB" gate="G$1" pin="D1"/>
-<wire x1="119.38" y1="119.38" x2="177.8" y2="119.38" width="0.1524" layer="91"/>
 </segment>
 </net>
@@
 <pinref part="C22" gate="G$1" pin="1"/>
 <pinref part="C28" gate="G$1" pin="2"/>
-<wire x1="137.16" y1="124.46" x2="147.32" y2="124.46" width="0.1524" layer="91"/>
+<wire x1="137.16" y1="124.46" x2="144.78" y2="124.46" width="0.1524" layer="91"/>
+<wire x1="144.78" y1="124.46" x2="147.32" y2="124.46" width="0.1524" layer="91"/>
 <wire x1="137.16" y1="127" x2="137.16" y2="124.46" width="0.1524" layer="91"/>
 <junction x="137.16" y="124.46"/>
-</segment>
-</net>
+<pinref part="RSNSI" gate="R1" pin="4"/>
+<wire x1="144.78" y1="149.86" x2="144.78" y2="124.46" width="0.1524" layer="91"/>
+<junction x="144.78" y="124.46"/>
+</segment>
+</net>
+<net name="D+1" class="0">
+<segment>
+<wire x1="274.32" y1="160.02" x2="276.86" y2="160.02" width="0.1524" layer="91"/>
+<wire x1="271.78" y1="165.1" x2="274.32" y2="165.1" width="0.1524" layer="91"/>
+<wire x1="274.32" y1="165.1" x2="274.32" y2="160.02" width="0.1524" layer="91"/>
+<wire x1="274.32" y1="160.02" x2="274.32" y2="152.4" width="0.1524" layer="91"/>
+<wire x1="274.32" y1="152.4" x2="276.86" y2="152.4" width="0.1524" layer="91"/>
+<junction x="274.32" y="160.02"/>
+<pinref part="R37" gate="G$1" pin="1"/>
+<pinref part="R38" gate="G$1" pin="1"/>
+<pinref part="CN5" gate="G$1" pin="D+"/>
+</segment>
+</net>
+<net name="D-1" class="0">
+<segment>
+<wire x1="274.32" y1="180.34" x2="276.86" y2="180.34" width="0.1524" layer="91"/>
+<wire x1="274.32" y1="172.72" x2="276.86" y2="172.72" width="0.1524" layer="91"/>
+<wire x1="274.32" y1="172.72" x2="274.32" y2="180.34" width="0.1524" layer="91"/>
+<wire x1="271.78" y1="167.64" x2="274.32" y2="167.64" width="0.1524" layer="91"/>
+<wire x1="274.32" y1="167.64" x2="274.32" y2="172.72" width="0.1524" layer="91"/>
+<junction x="274.32" y="172.72"/>
+<pinref part="R35" gate="G$1" pin="1"/>
+<pinref part="R36" gate="G$1" pin="1"/>
+<pinref part="CN5" gate="G$1" pin="D-"/>
+</segment>
+</net>
+<net name="N$2" class="0">
+<segment>
+<pinref part="U1" gate="A" pin="SYSM5"/>
+<pinref part="C30" gate="G$1" pin="2"/>
+<wire x1="119.38" y1="119.38" x2="134.62" y2="119.38" width="0.1524" layer="91"/>
+</segment>
+</net>
+<net name="N$4" class="0">
+<segment>
+<pinref part="C30" gate="G$1" pin="1"/>
+<pinref part="M3AB" gate="G$1" pin="D1"/>
+<wire x1="142.24" y1="119.38" x2="177.8" y2="119.38" width="0.1524" layer="91"/>
+</segment>
+</net>
